File: EMG_Amplifier_board/EMG_acquisition_module_panel.kicad_pcb (KiCad board)
At the start: 2 copper layers, 52 x 30 mm, 50 parts, among them J1 Conn_01x04_Socket, J2 Conn_01x04_Pin, J3 Conn_01x06_Pin, J4 Conn_01x06_Socket, J7 Conn_01x06_Pin, U1 LPV821DBVR, U2 INA333xxDGK, U3 LPV821DBVR, U5 LPV821DBVR, U6 LPV821DBVR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

Commit message: place all components on one side
Parts:
- C10, C11, C12, R23, R24: moved to B.Cu
- moved R19 4.09 mm to (86.4, 108.4)
- moved R12 2.94 mm to (94.7, 108.1), turned to 0 degrees
- moved R10 2.87 mm to (75.2, 108.0)
- moved C4 2.75 mm to (72.1, 108.3)
- moved R13 2.75 mm to (91.5, 108.1), turned to 180 degrees
- moved R22 2.34 mm to (77.4, 106.1)
- moved C6 2.33 mm to (88.8, 107.4), turned to -90 degrees
- moved R11 2.21 mm to (74.7, 106.1)
- moved C3 2.02 mm to (76.0, 106.1)
- moved R21 1.98 mm to (75.2, 104.2)
- moved R24 1.34 mm to (90.5, 98.7)
- moved R23 1.26 mm to (88.8, 97.3), turned to -90 degrees
- moved C11 1.15 mm to (94.4, 108.0)
- moved U2 0.58 mm to (93.0, 105.4)
- moved U6 0.48 mm to (85.4, 96.8)
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Routing:
- net GND: track 56.9 -> 65.4 mm, vias 21 -> 19
- net /Filtering_Board/V_PR: track 32.5 -> 28.5 mm
- net /Processing_Board/LPF_400Hz/V_EMG_INA: track 19.8 -> 16.5 mm, vias 2 -> 0
- net /Processing_Board/V_CM: track 15.3 -> 12.5 mm
- net /Processing_Board/V_EMG_OUT: track 10.8 -> 13.1 mm
- net Net-(U2-Ref): track 12.9 -> 11.1 mm, vias 0 -> 3
- net /Filtering_Board/+V_DD: track 71.1 -> 69.5 mm
- net Net-(U3-IN+): track 12.6 -> 11.0 mm
- net +1V8: track 85.7 -> 84.2 mm, vias 10 -> 5
- net Net-(U8--INB): track 7.55 -> 6.28 mm
- net Net-(U6-IN+): track 8.91 -> 7.69 mm, vias 0 -> 1
- net Net-(U3-IN-): track 9.57 -> 8.79 mm
- net Net-(U1-IN-): track 3.38 -> 4.14 mm
- net Net-(U6-IN-): track 11.1 -> 10.4 mm
- net Net-(C4-Pad1): track 3.72 -> 3.15 mm
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