File: EMG_Amplifier_board/DRL.kicad_sch (KiCad schematic)
At the start: 8 parts, among them U5 LPV821DBVR, U6 LPV821DBVR

Commit message: update R and C refs to correspond to paper
Parts:
- renumbered C9 to C21, C8 to C22, R23 to R31, R24 to R32
Changed lines of the file:
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@@
 	(wire
 		(pts
-			(xy 110.49 49.53) (xy 69.85 49.53)
+			(xy 110.49 49.53) (xy 105.41 49.53)
 		)
 		(stroke
@@
 		(dnp no)
 		(fields_autoplaced yes)
-		(property "Reference" "C9"
-			(at 148.5963 44.45 90)
+		(property "Reference" "C21"
+			(at 148.5963 31.75 90)
 			(effects
 				(font
@@
 		)
 		(property "Value" "0.1uF"
-			(at 148.5963 41.91 90)
+			(at 148.5963 34.29 90)
 			(effects
 				(font
@@
 			(project "EMG_amplifier"
 				(path "/26861adc-1ddf-4c37-9f8b-8db1c0839771/566a5450-97e0-4bc1-8c47-b0ac1397ab98/87e3490f-ae1c-443c-8c09-d2b58f9f3cb7"
-					(reference "C9")
+					(reference "C21")
 					(unit 1)
 				)
@@
 	(symbol
 		(lib_id "power:GND")
-		(at 69.85 49.53 270)
+		(at 105.41 49.53 270)
 		(mirror x)
 		(unit 1)
@@
 		(on_board yes)
 		(dnp no)
-		(fields_autoplaced yes)
 		(property "Reference" "#PWR017"
-			(at 63.5 49.53 0)
+			(at 99.06 49.53 0)
 			(effects
 				(font
@@
 		)
 		(property "Value" "GND"
-			(at 66.04 49.5299 90)
+			(at 101.6 49.5299 90)
 			(effects
 				(font
@@
 		)
 		(property "Footprint" ""
-			(at 69.85 49.53 0)
+			(at 105.41 49.53 0)
 			(effects
 				(font
@@
 		)
 		(property "Datasheet" ""
-			(at 69.85 49.53 0)
+			(at 105.41 49.53 0)
 			(effects
 				(font
@@
 		)
 		(property "Description" "Power symbol creates a global label with name \"GND\" , ground"
-			(at 69.85 49.53 0)
+			(at 105.41 49.53 0)
 			(effects
 				(font
@@
 		(dnp no)
 		(fields_autoplaced yes)
-		(property "Reference" "C8"
-			(at 165.1 76.1937 90)
-			(effects
-				(font
-					(size 1.27 1.27)
-				)
+		(property "Reference" "C22"
+			(at 156.21 74.9235 0)
+			(effects
+				(font
+					(size 1.27 1.27)
+				)
+				(justify right)
 			)
 		)
 		(property "Value" "0.1uF"
-			(at 162.56 76.1937 90)
-			(effects
-				(font
-					(size 1.27 1.27)
-				)
+			(at 156.21 77.4635 0)
+			(effects
+				(font
+					(size 1.27 1.27)
+				)
+				(justify right)
 			)
 		)
@@
 			(project "EMG_amplifier"
 				(path "/26861adc-1ddf-4c37-9f8b-8db1c0839771/566a5450-97e0-4bc1-8c47-b0ac1397ab98/87e3490f-ae1c-443c-8c09-d2b58f9f3cb7"
-					(reference "C8")
+					(reference "C22")
 					(unit 1)
 				)
@@
 		(dnp no)
 		(fields_autoplaced yes)
-		(property "Reference" "R23"
+		(property "Reference" "R31"
 			(at 128.27 43.18 90)
 			(effects
@@
 			(project ""
 				(path "/26861adc-1ddf-4c37-9f8b-8db1c0839771/566a5450-97e0-4bc1-8c47-b0ac1397ab98/87e3490f-ae1c-443c-8c09-d2b58f9f3cb7"
-					(reference "R23")
+					(reference "R31")
 					(unit 1)
 				)
@@
 		(dnp no)
 		(fields_autoplaced yes)
-		(property "Reference" "R24"
+		(property "Reference" "R32"
 			(at 114.3 43.18 90)
 			(effects
@@
 			(project ""
 				(path "/26861adc-1ddf-4c37-9f8b-8db1c0839771/566a5450-97e0-4bc1-8c47-b0ac1397ab98/87e3490f-ae1c-443c-8c09-d2b58f9f3cb7"
-					(reference "R24")
+					(reference "R32")
 					(unit 1)
 				)

Commit message: replace 2012 capacitors with 1005
Parts:
- C21, C22: footprint Capacitor_SMD:C_0805_2012Metric -> Capacitor_SMD:C_0402_1005Metric
Changed lines of the file:
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@@
 			)
 		)
-		(property "Footprint" "Capacitor_SMD:C_0805_2012Metric"
+		(property "Footprint" "Capacitor_SMD:C_0402_1005Metric"
 			(at 148.59 38.1 0)
 			(effects
@@
 			)
 		)
-		(property "Footprint" "Capacitor_SMD:C_0805_2012Metric"
+		(property "Footprint" "Capacitor_SMD:C_0402_1005Metric"
 			(at 158.75 76.2 0)
 			(effects
