File: EMG_Amplifier_board/DRL.kicad_sch (KiCad schematic)
At the start: 8 parts, among them U5 LPV821DBVR, U6 LPV821DBVR

Commit message: minor changes
Parts:
- U5, U6: footprint SOT95P280X145-5N -> LPV821DBVR:SOT95P280X145-5N
Changed lines of the file:
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@@
 			)
 		)
-		(property "Footprint" "SOT95P280X145-5N"
+		(property "Footprint" "LPV821DBVR:SOT95P280X145-5N"
 			(at 180.34 93.98 0)
 			(effects
@@
 			)
 		)
-		(property "Footprint" "SOT95P280X145-5N"
+		(property "Footprint" "LPV821DBVR:SOT95P280X145-5N"
 			(at 107.95 91.44 0)
 			(effects

Commit message: add buck converter 3v3 to 1v8, start new two-board sigacq project
Parts:
- U5, U6: footprint LPV821DBVR:SOT95P280X145-5N -> Package_TO_SOT_SMD:SOT-23-5
Changed lines of the file:
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@@
 			)
 		)
-		(property "Footprint" "LPV821DBVR:SOT95P280X145-5N"
+		(property "Footprint" "Package_TO_SOT_SMD:SOT-23-5"
 			(at 180.34 93.98 0)
 			(effects
@@
 			)
 		)
-		(property "Footprint" "LPV821DBVR:SOT95P280X145-5N"
+		(property "Footprint" "Package_TO_SOT_SMD:SOT-23-5"
 			(at 107.95 91.44 0)
 			(effects
