File: EMG_Amplifier_board/LPF_400Hz.kicad_sch (KiCad schematic)
At the start: 6 parts, among them U1 LPV821DBVR

Commit message: replace 2012 capacitors with 1005
Parts:
- C23: footprint Capacitor_SMD:C_0805_2012Metric -> Capacitor_SMD:C_0402_1005Metric
Changed lines of the file:
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@@
 			)
 		)
-		(property "Footprint" "Capacitor_SMD:C_0805_2012Metric"
+		(property "Footprint" "Capacitor_SMD:C_0402_1005Metric"
 			(at 177.8 76.2 0)
 			(effects

Commit message: minor changes
Parts:
- U1: footprint Components:SOT95P280X145-5N -> LPV821DBVR:SOT95P280X145-5N
Changed lines of the file:
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@@
 			)
 		)
-		(property "Footprint" "Components:SOT95P280X145-5N"
+		(property "Footprint" "LPV821DBVR:SOT95P280X145-5N"
 			(at 148.59 93.98 0)
 			(effects

Commit message: add buck converter 3v3 to 1v8, start new two-board sigacq project
Parts:
- U1: footprint LPV821DBVR:SOT95P280X145-5N -> Package_TO_SOT_SMD:SOT-23-5
Changed lines of the file:
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@@
 			)
 		)
-		(property "Footprint" "LPV821DBVR:SOT95P280X145-5N"
+		(property "Footprint" "Package_TO_SOT_SMD:SOT-23-5"
 			(at 148.59 93.98 0)
 			(effects
